File: Hardware/mailbox.sch (EAGLE design)
At the start: 24 parts, among them U3 V_REG_LDOSMD, U5 MCP73831

Commit message: Added battery measure + PDF schematic
Parts:
- removed C1: 100nF, SparkFun-Passives:CAP0402-CAP
- removed C3: 10uF, SparkFun-Passives:CAP0402-CAP
- removed D4: Yellow, SparkFun-LED:LED-YELLOW0603
- removed R4, R5, R6: 10K, SparkFun-Passives:RESISTOR0402-RES
- added C4, C5: 10uF, SparkFun-Passives:CAP1206
- added D6: YELLOW, SparkFun-LED:LED-YELLOW1206
- added R10, R13, R9: 10K, SparkFun-Passives:RESISTOR1206
- added R7: 1M, SparkFun-Passives:RESISTOR1206
- added R8: 220, SparkFun-Passives:RESISTOR1206
- C2: value 10uF -> 100nF; device SparkFun-Passives:CAP0402-CAP -> SparkFun-Passives:CAP1206
- R1: value 10K -> 1K; device SparkFun-Passives:RESISTOR0402-RES -> SparkFun-Passives:RESISTOR1206
- R11: value 2K -> 10K; device SparkFun-Passives:RESISTOR0603-RES -> SparkFun-Passives:RESISTOR1206
- R12: value 1K -> 10K; device SparkFun-Passives:RESISTOR0603-RES -> SparkFun-Passives:RESISTOR1206
- R2: value 10K -> 2K; device SparkFun-Passives:RESISTOR0402-RES -> SparkFun-Passives:RESISTOR1206
- R3: device SparkFun-Passives:RESISTOR0402-RES -> SparkFun-Passives:RESISTOR1206
Connections:
- net 3.3V: now also C5.1, R10.2, R12.2, R3.2, R9.2; no longer C3.1, R1.2, R2.2, R4.2, R5.2
- net ADC: now also R7.1, R8.2
- net CH_PD: now also C2.1, R10.1; no longer C1.2, R2.1
- net GND: now also C4.2, C5.2, R13.1, R2.2, R8.1; no longer C2.2, C3.2, R11.2, R6.1
- net GPIO0: now also R9.1; no longer R1.1
- net GPIO15: now also R13.2; no longer R6.2
- net GPIO2: now also R12.1; no longer R5.1
- net LDO_EN: now also R11.1; no longer R3.1
- net N$1: now also D6.C, R1.1; no longer D4.C, R12.1
- net N$3: now also C2.2; no longer C1.1
- net N$6: now also R1.2; no longer R12.2
- net N$7: now also R2.1; no longer R11.1
- net RESET: now also R3.1; no longer R4.1
- net V_BATT: now also R7.2
- net V_USB: now also C4.1, D6.A, R11.2; no longer C2.1, D4.A, R3.2
Other:
- note added: "Batt. Measure"
- note removed: "D1,D2,D3 - B5819W R1,R2 - 10K C1 - 100nf"
- moved on the sheet: C2, R1, R11, R12, R2, R3
